Commit message: 虚拟小车完成

File: src/velodyne_simulator/velodyne_description/urdf/Scout_base.urdf.xacro (robot description, xacro)
@@ -5,4 +5,16 @@
   <xacro:arg name="organize_cloud" default="false"/>
   <xacro:property name="organize_cloud" value="$(arg organize_cloud)" />
+ <!-- 属性封装 -->
+  <xacro:property name="M_PI" value="3.14159"/>
+  <xacro:property name="base_x_size" value="0.9250000" />
+  <xacro:property name="base_y_size" value="0.380000" />
+  <xacro:property name="base_z_size" value="0.210000" />
+  <xacro:property name="wheelbase" value="0.498" />
+  <xacro:property name="track" value="0.58306" />   <!-- track车轮间距 -->
+  <xacro:property name="wheel_vertical_offset" value="-0.0702" />
+  <xacro:property name="wheel_length" value="1.1653e-01" />
+  <xacro:property name="wheel_radius" value="1.6459e-01" />
+  <xacro:property name="footprint_hight" value="0.234845" />
+  <xacro:include filename="$(find velodyne_description)/urdf/inertial.xacro"/>    <!-- 引用惯性矩阵计算 -->
   <!-- Base Footprint -->
   <link name="base_footprint" />
@@ -11,25 +23,64 @@
    <parent link="base_footprint" />
     <child link="base_link" />
-    <origin xyz="0 0 0.05" rpy="0 0 0" />
+    <origin xyz="0 0 ${footprint_hight}" rpy="0 0 0" />
   </joint>
   <link name="base_link" >
-    <visual>
-      <geometry>
-        <box size="0.5 0.5 0.1" />
-      </geometry>
+  <visual>
+        <origin xyz="0 0 0" rpy="0 0 0" />
+        <geometry>
+            <mesh filename="package://velodyne_description/meshes/Scout_meshes/base_link.dae" />
+        </geometry>
     </visual>
-    <collision>
-      <geometry>
-        <box size="0.5 0.5 0.1" />
-      </geometry>
+ <collision>
+        <origin xyz="0 0 0.008" rpy="0 0 0" />
+        <geometry>
+            <box size="${base_x_size} ${base_y_size} ${base_z_size}"/>
+        </geometry>
     </collision>
-    <inertial>
-      <origin xyz="0 0 0"/>
-      <mass value="10"/>
-      <inertia ixx="3.0" ixy="0.0" ixz="0.0"
-               iyy="3.0" iyz="0.0"
-               izz="3.0" />
-    </inertial>
+        <collision>
+        <origin xyz="0 0 ${base_z_size/6}" rpy="0 0 0" />
+        <geometry>
+            <box size="${base_x_size/6} ${base_y_size*1.65} ${base_z_size/3}"/>
+        </geometry>
+    </collision>
+            <inertial>
+            <mass value="40" />
+            <origin xyz="0.0 0.0 0.0" />
+            <inertia ixx="2.288641" ixy="0" ixz="0" iyy="5.103976" iyz="0" izz="3.431465" />
+        </inertial>
   </link>
+  <!-- 雷达支架 -->
+  <xacro:property name="support_length" value="0.30" /> <!-- 支架长度 -->
+  <xacro:property name="support_radius" value="0.025" /> <!-- 支架半径 -->
+  <xacro:property name="support_x_size" value="0.0" /> <!-- 支架安装的x坐标 -->
+  <xacro:property name="support_y_size" value="0.0" /> <!-- 支架安装的y坐标 -->
+  <xacro:property name="support_z_size" value="${base_z_size / 2 + support_length / 2}" /> <!-- 支架安装的z坐标:底盘高度 / 2 + 支架高度 / 2  -->
+  <xacro:property name="support_m" value="0.02" /> <!-- 支架质量 -->
+  <link name="support">
+      <visual>
+          <geometry>
+              <cylinder radius="${support_radius}" length="${support_length}" />
+          </geometry>
+          <origin xyz="0.0 0.0 0.0" rpy="0.0 0.0 0.0" />
+          <material name="red">
+              <color rgba="0.8 0.2 0.0 0.8" />
+          </material>
+      </visual>
+      <collision>
+          <geometry>
+              <cylinder radius="${support_radius}" length="${support_length}" />
+          </geometry>
+          <origin xyz="0.0 0.0 0.0" rpy="0.0 0.0 0.0" />
+      </collision>
+      <xacro:cylinder_inertial_matrix m="${support_m}" r="${support_radius}" h="${support_length}" />
+  </link>
+  <joint name="support_2_base_link" type="fixed">
+      <parent link="base_link" />
+      <child link="support" />
+      <origin xyz="${support_x_size} ${support_y_size} ${support_z_size}" />
+  </joint>
+  <gazebo reference="support">
+      <material>Gazebo/White</material>
+  </gazebo>
   <!-- 引用激光雷达 -->
   <xacro:include filename="$(find velodyne_description)/urdf/VLP-16.urdf.xacro"/>
@@ -37,3 +88,22 @@
     <origin xyz="0 0 0.4" rpy="0 0 0" />
   </xacro:VLP-16>
+  <!-- 引用车轮 -->
+  <xacro:include filename="$(find velodyne_description)/urdf/scout_wheel_type1.xacro" />
+  <xacro:include filename="$(find velodyne_description)/urdf/scout_wheel_type2.xacro" />
+  <xacro:scout_wheel_type1 wheel_prefix="front_right">
+      <origin xyz="${wheelbase/2} ${-track/2} ${wheel_vertical_offset}" rpy="3.14 0 0" />
+  </xacro:scout_wheel_type1>
+  <xacro:scout_wheel_type2 wheel_prefix="front_left">
+      <origin xyz="${wheelbase/2} ${track/2} ${wheel_vertical_offset}" rpy="0 0 0" />
+  </xacro:scout_wheel_type2>
+  <xacro:scout_wheel_type1 wheel_prefix="rear_left">
+      <origin xyz="${-wheelbase/2} ${track/2} ${wheel_vertical_offset}" rpy="0 0 0" />
+  </xacro:scout_wheel_type1>
+  <xacro:scout_wheel_type2 wheel_prefix="rear_right">
+      <origin xyz="${-wheelbase/2} ${-track/2} ${wheel_vertical_offset}" rpy="3.14 0 0" />
+  </xacro:scout_wheel_type2>
+  <!-- 引用控制插件 -->
+  <xacro:include filename="$(find velodyne_description)/urdf/move.xacro"/>
+  <!-- 引用imu插件 -->
+  <xacro:include filename="$(find velodyne_description)/urdf/imu.xacro"/>
 </robot>
